File: Project/KiCad/Sporbesat-Detektor/Sporbesat-Detektor.kicad_sch (KiCad schematic)
At the start: 18 parts, among them J1 Screw_Terminal_01x02, J2 Screw_Terminal_01x02, J3 Conn_01x05_Socket, Q1 BC857, U1 4N35

Commit message: Test Board
Parts:
- removed U1: 4N35, Package_DIP:DIP-6_W7.62mm, symbol Isolator:4N35
- added U1: PC847, Package_DIP:DIP-16_W7.62mm, symbol Isolator:PC847
- C1: value ?F -> 200nF
Connections:
- net GNDD: now also U1.15
- net GNDDCC: now also U1.2
- net at D4.1 (K): now also U1.1
- net at D5.1 (K), J3.1 (Pin_1): now also U1.16
Other:
- moved on the sheet: D5, J3, R5
