File: Project/Sikring/Sporbesat/Sikring_Sporbesat/Sikring_Sporbesat2.kicad_sch (KiCad schematic)
At the start: 20 parts, among them J1 Screw_Terminal_01x02, J2 Screw_Terminal_01x02, Q1 BC857, Q2 BC847, U1 PC847

Commit message: Beskrivelse af functionen af Sporbesat detektor
Parts:
- C2: value 47nF -> 22nF
Changed lines of the file:
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@@
 			)
 		)
-		(property "Value" "47nF"
+		(property "Value" "22nF"
 			(at 151.638 63.5 0)
 			(show_name no)

Commit message: ændringer efter test 20261017
Parts:
- added C3: 100nF, symbol Device:C
- C2: value 22nF -> 100nf
- R1: value 10Ω -> 1KΩ
Connections:
- net VDCC: now also C3.1
- net VTRACK: now also C3.2
Other:
- moved on the sheet: C1, C2, D1, D2, D3, D4, D5, J1, J2, Q1, Q2, R1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
