File: Project/Sikring/Sporbesat/Sikring_Sporbesat/Sikring_Sporbesat2.kicad_sch (KiCad schematic)
At the start: 21 parts, among them J1 Screw_Terminal_01x02, J2 Screw_Terminal_01x02, Q1 BC857, Q2 BC847, U1 PC847

Commit message: sporbesat tegnibńger
Parts:
- added RV1: 200K, Valve:Valve_Noval_P, symbol Device:R_Potentiometer_Small
- C2: value 100nf -> 22nf
Connections:
- net at C2.1, D4.1 (K), R4.1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: now also RV1.1; no longer R2.2
- new net: R2.2, RV1.2, RV1.3
Other:
- moved on the sheet: C2, D4, R2, R4, TP2
