File: Project/Sikring/Sporbesat/Sikring_Sporbesat/Sikring_Sensor.kicad_sch (KiCad schematic)
At the start: 61 parts, among them Q1 BC857, Q2 BC847, Q3 BC857, Q4 BC847, Q5 BC857, Q6 BC847, Q7 BC857, Q8 BC847, U1 PC847

Commit message: NYT PCB
Parts:
- added H1, H2, H3, H4: MountingHole_Pad, MountingHole:MountingHole_3.2mm_M3_Pad_TopBottom, symbol Mechanical:MountingHole_Pad
- added J3: Conn_01x05_Pin, Connector_Molex:Molex_SL_171971-0005_1x05_P2.54mm_Vertical, symbol Connector:Conn_01x05_Pin
Connections:
- net GDIGI: now also H1.1, H2.1, H3.1, H4.1, J3.5 (Pin_5)
- net BESAT1: no longer names the net of U1.16
- net BESAT1: now also J3.1 (Pin_1)
- net BESAT2: no longer names the net of U1.14
- net BESAT2: now also J3.2 (Pin_2)
- net BESAT3: no longer names the net of U1.12
- net BESAT3: now also J3.3 (Pin_3)
- net BESAT4: no longer names the net of U1.10
- net BESAT4: now also J3.4 (Pin_4)
